File: SmartyB-hw/SmartyB-hw.kicad_pcb (KiCad board)
At the start: 2 copper layers, 80 x 80 mm, 20 parts, among them J1 1-2071556-2, J2 1-2071556-2, J3 Screw_Terminal_01x03, J4 Screw_Terminal_01x03, Q1 Q_NMOS_DGS, Q2 Q_NMOS_DGS, SW1 SW_Push, SW2 SW_Push, SW3 SW_Push, SW4 SW_Push

Commit message: hw gerbers
Routing:
- net GND: track 110.0 -> 111.7 mm, vias 0 -> 2
Changed lines of the file:
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@@
 			(outputformat 1)
 			(mirror no)
-			(drillshape 1)
+			(drillshape 0)
 			(scaleselection 1)
-			(outputdirectory "")
+			(outputdirectory "SmartyB-hw-backups/")
 		)
 	)
@@
 		(net 7)
 	)
+	(via
+		(at 75.5 76)
+		(size 2)
+		(drill 1)
+		(layers "F.Cu" "B.Cu")
+		(net 8)
+	)
+	(via
+		(at 58.5 93)
+		(size 2)
+		(drill 1)
+		(layers "F.Cu" "B.Cu")
+		(net 8)
+	)
 	(segment
 		(start 50 88)
@@
 	)
 	(segment
-		(start 93 95.54)
-		(end 76.54 95.54)
+		(start 60.5 95)
+		(end 76 95)
+		(width 1)
+		(layer "B.Cu")
+		(net 8)
+	)
+	(segment
+		(start 75.5 76)
+		(end 71.18 80.32)
+		(width 1)
+		(layer "B.Cu")
+		(net 8)
+	)
+	(segment
+		(start 56.5 95)
+		(end 48.54 95)
 		(width 1)
 		(layer "B.Cu")
@@
 	(segment
 		(start 82.5325 68.9675)
-		(end 71.18 80.32)
+		(end 75.5 76)
 		(width 1)
 		(layer "B.Cu")
@@
 	)
 	(segment
-		(start 76 95)
-		(end 48.54 95)
+		(start 36.5 94.04)
+		(end 39.77 97.31)
 		(width 1)
 		(layer "B.Cu")
@@
 	)
 	(segment
-		(start 36.5 94.04)
-		(end 39.77 97.31)
+		(start 76.54 95.54)
+		(end 93 95.54)
+		(width 1)
+		(layer "B.Cu")
+		(net 8)
+	)
+	(segment
+		(start 76 95)
+		(end 76.54 95.54)
 		(width 1)
 		(layer "B.Cu")
@@
 	)
 	(segment
-		(start 76.54 95.54)
-		(end 76 95)
+		(start 58.5 93)
+		(end 60.5 95)
 		(width 1)
 		(layer "B.Cu")
@@
 		(width 1)
 		(layer "B.Cu")
+		(net 8)
+	)
+	(segment
+		(start 58.5 93)
+		(end 56.5 95)
+		(width 1)
+		(layer "B.Cu")

Commit message: hw minor adjustment
Parts:
- moved J1 2.73 mm to (43.3, 49.2)
- moved J2 2.73 mm to (43.3, 36.8)
- moved SW1 2.25 mm to (98.2, 59.5)
- moved SW2 2.25 mm to (91.8, 73.5)
- moved SW3 2.25 mm to (55.2, 59.5)
- moved SW4 2.25 mm to (48.8, 73.5)
- moved J3 0.50 mm to (91.0, 50.0)
Routing:
- net +5V: track 106.3 -> 93.2 mm
- net +3V3: track 74.8 -> 80.6 mm
- net /AC_IN_L: track 57.7 -> 54.1 mm
- net /AC_SW2_L: track 47.6 -> 44.4 mm
- net /AC_SW1_L: track 38.3 -> 35.2 mm
- net /BTN3: track 61.0 -> 64.1 mm
- net Net-(J2-COIL_2): track 63.8 -> 66.6 mm
- net /BTN1: track 38.9 -> 41.3 mm
- net /BTN4: track 50.6 -> 49.5 mm
- net /SW2: track 43.2 -> 44.2 mm
- net /SW1: track 26.7 -> 27.7 mm
- net /BTN2: track 18.0 -> 17.1 mm
- net Net-(J1-COIL_2): track 55.0 -> 54.2 mm
Other:
- outline, holes or cut-outs redrawn
