File: SmartyB-hw/SmartyB-hw.kicad_pcb (KiCad board)
At the start: 2 copper layers, 80 x 80 mm, 20 parts, among them J1 1-2071556-2, J2 1-2071556-2, J3 Screw_Terminal_01x03, J4 Screw_Terminal_01x03, Q1 Q_NMOS_DGS, Q2 Q_NMOS_DGS, SW1 SW_Push, SW2 SW_Push, SW3 SW_Push, SW4 SW_Push

Commit message: hw revisionssss
Routing:
- net /BTN1: track 41.3 -> 45.9 mm
- net Net-(J2-COIL_2): track 66.6 -> 65.0 mm
Other:
- outline, holes or cut-outs redrawn

Commit message: hw revisionssss2
Parts:
- moved J3 0.50 mm to (91.0, 49.5)
Routing:
- net GND: track 111.2 -> 140.8 mm
- net +3V3: track 80.2 -> 106.2 mm
- net /BTN1: track 45.9 -> 53.0 mm
- net /BTN4: track 49.5 -> 56.0 mm
- net /BTN3: track 63.7 -> 70.2 mm
- net /BTN2: track 17.1 -> 23.6 mm
- net /AC_IN_L: track 54.1 -> 50.0 mm
- net /AC_SW2_L: track 44.4 -> 45.8 mm
Other:
- outline, holes or cut-outs redrawn
Changed lines of the file:
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@@
 		(tags "Connector")
 		(property "Reference" "J1"
-			(at 7.93 -3.8 0)
+			(at 7.43 -3.3 0)
 			(layer "F.SilkS")
 			(effects
@@
 		)
 		(fp_text user "${REFERENCE}"
-			(at 7.93 -3.8 0)
+			(at 7.43 -3.3 0)
 			(layer "F.Fab")
 			(effects
@@
 		(tags "Connector")
 		(property "Reference" "J2"
-			(at 7.93 -3.8 0)
+			(at 7.43 -3.3 0)
 			(layer "F.SilkS")
 			(effects
@@
 		)
 		(fp_text user "${REFERENCE}"
-			(at 7.93 -3.8 0)
+			(at 7.43 -3.3 0)
 			(layer "F.Fab")
 			(effects
@@
 	(footprint "TerminalBlock_RND:TerminalBlock_RND_205-00046_1x03_P5.00mm_Horizontal"
 		(layer "F.Cu")
-		(at 91 50 90)
+		(at 91 49.5 90)
 		(descr "terminal block RND 205-00046, 3 pins, pitch 5mm, size 15x8.1mm, drill diameter 1.1mm, pad diameter 2.1mm, http://cdn-reichelt.de/documents/datenblatt/C151/RND_205-00045_DB_EN.pdf, script-generated using https://gitlab.com/kicad/libraries/kicad-footprint-generator/-/tree/master/scripts/TerminalBlock_RND")
 		(tags "THT terminal block RND 205-00046 pitch 5mm size 15x8.1mm drill 1.1mm pad 2.1mm")
@@
 	)
 	(gr_line
-		(start 51.5 31)
-		(end 51.5 47.75)
+		(start 51 30)
+		(end 51 49.5)
 		(stroke
 			(width 0.05)
@@
 	)
 	(gr_line
-		(start 49.5 31)
-		(end 49.5 47.75)
+		(start 49 30)
+		(end 49 49.5)
 		(stroke
 			(width 0.05)
@@
 	)
 	(gr_arc
-		(start 49.5 31)
-		(mid 50.5 30)
-		(end 51.5 31)
+		(start 49 30)
+		(mid 50 29)
+		(end 51 30)
 		(stroke
 			(width 0.05)
@@
 	)
 	(gr_arc
-		(start 51.5 47.75)
-		(mid 50.5 48.75)
-		(end 49.5 47.75)
+		(start 51 49.5)
+		(mid 50 50.5)
+		(end 49 49.5)
 		(stroke
 			(width 0.05)
@@
 	)
 	(segment
-		(start 56.499 49.499)
-		(end 91 49.499)
-		(width 2)
+		(start 90.751 49.749)
+		(end 91 49.5)
+		(width 2.5)
+		(layer "B.Cu")
+		(net 1)
+	)
+	(segment
+		(start 56.749 49.749)
+		(end 90.751 49.749)
+		(width 2.5)
 		(layer "B.Cu")
 		(net 1)
@@
 	(segment
 		(start 56 49)
-		(end 56.499 49.499)
-		(width 2)
+		(end 56.749 49.749)
+		(width 2.5)
 		(layer "B.Cu")
 		(net 1)
 	)
 	(segment
-		(start 58.54 29.4)
-		(end 60.5 31.36)
-		(width 2)
+		(start 90 40.5)
+		(end 59.94 40.5)
+		(width 2.5)
 		(layer "B.Cu")
 		(net 2)
 	)
 	(segment
-		(start 91 40)
-		(end 60.44 40)
-		(width 2)
+		(start 59.9 40.54)
+		(end 59.9 30.76)
+		(width 2.5)
 		(layer "B.Cu")
 		(net 2)
 	)
 	(segment
-		(start 60.5 39.94)
-		(end 58.54 41.9)
-		(width 2)
+		(start 59.9 30.76)
+		(end 58.54 29.4)
+		(width 2.5)
 		(layer "B.Cu")
 		(net 2)
 	)
 	(segment
-		(start 60.5 31.36)
-		(end 60.5 39.94)
-		(width 2)
+		(start 91 39.5)
+		(end 90 40.5)
+		(width 2.5)
 		(layer "B.Cu")
 		(net 2)
@@
 		(start 64.7525 30.76)
 		(end 59.9 30.76)
-		(width 2)
+		(width 2.5)
 		(layer "B.Cu")
 		(net 2)
 	)
 	(segment
-		(start 60.44 40)
-		(end 58.54 41.9)
-		(width 2)
+		(start 59.94 40.5)
+		(end 59.9 40.54)
+		(width 2.5)
 		(layer "B.Cu")
 		(net 2)
 	)
 	(segment
-		(start 59.9 30.76)
-		(end 58.54 29.4)
-		(width 2)
+		(start 58.54 41.9)
+		(end 59.9 40.54)
+		(width 2.5)
 		(layer "B.Cu")
 		(net 2)
@@
 	)
 	(segment
-		(start 54.5 38)
-		(end 54.5 43)
+		(start 61.96301 45.53699)
+		(end 62.5 45)
 		(width 2)
 		(layer "B.Cu")
@@
 	)
 	(segment
-		(start 56.5 45)
-		(end 91 45)
+		(start 54 38.5)
+		(end 54 43.055864)
 		(width 2)
 		(layer "B.Cu")
@@
 	)
 	(segment
-		(start 56 36.5)
-		(end 54.5 38)
-		(width 2)
+		(start 90.5 45)
+		(end 62.5 45)
+		(width 2.5)
 		(layer "B.Cu")
 		(net 6)
 	)
 	(segment
-		(start 54.5 43)
-		(end 56.5 45)
+		(start 54 43.055864)
+		(end 56.481126 45.53699)
 		(width 2)
 		(layer "B.Cu")
@@
 	)
 	(segment
-		(start 100.5 31)
-		(end 75.5 31)
+		(start 54 38.5)
+		(end 56 36.5)
+		(width 2.5)
+		(layer "B.Cu")
+		(net 6)
+	)
+	(segment
+		(start 56.481126 45.53699)
+		(end 61.96301 45.53699)
 		(width 2)
 		(layer "B.Cu")
+		(net 6)
+	)
+	(segment
+		(start 91 44.5)
+		(end 90.5 45)
+		(width 2.5)
+		(layer "B.Cu")
+		(net 6)
+	)
+	(segment
+		(start 83.5 31)
+		(end 78.666532 35.833468)
+		(width 2.5)
+		(layer "B.Cu")
 		(net 7)
 	)
 	(segment
-		(start 110.5 31)
-		(end 100.5 31)
-		(width 2)
+		(start 64.759032 35.833468)
+		(end 64.7525 35.84)
+		(width 2.5)
 		(layer "B.Cu")
 		(net 7)
 	)
 	(segment
-		(start 75.5 31)
-		(end 70.66 35.84)
-		(width 2)
+		(start 110.5 31)
+		(end 83.5 31)
+		(width 2.5)
 		(layer "B.Cu")
 		(net 7)
 	)
 	(segment
-		(start 70.66 35.84)
-		(end 64.7525 35.84)
-		(width 2)
+		(start 78.666532 35.833468)
+		(end 64.759032 35.833468)
+		(width 2.5)
 		(layer "B.Cu")
 		(net 7)
 	)
+	(segment
+		(start 78 71.5)
+		(end 58.5 91)
+		(width 1)
+		(layer "F.Cu")
+		(net 8)
+	)
+	(segment
+		(start 58.5 91)
+		(end 58.5 93)
+		(width 1)
+		(layer "F.Cu")
+		(net 8)
+	)
 	(via
 		(at 78 71.5)
@@
 	)
 	(segment
+		(start 91.75 55)
+		(end 98.25 55)
+		(width 1)
+		(layer "F.Cu")
+		(net 12)
+	)
+	(segment
 		(start 95 78.75)
 		(end 89 84.75)
@@
 	)
 	(segment
+		(start 92.46 90.46)
+		(end 88.96 86.96)
+		(width 1)
+		(layer "B.Cu")
+		(net 12)
+	)
+	(segment
 		(start 95 58.25)
-		(end 98.25 55)
+		(end 95 55)
 		(width 1)
 		(layer "B.Cu")
@@
 	)
 	(segment
-		(start 92.46 90.46)
-		(end 88.96 86.96)
+		(start 95 55)
+		(end 98.25 55)
 		(width 1)
 		(layer "B.Cu")
@@
 	)
 	(segment
-		(start 88.96 86.96)
-		(end 88.96 86)
+		(start 95 55)
+		(end 91.75 55)
 		(width 1)
 		(layer "B.Cu")
@@
 	)
 	(segment
-		(start 95 58.25)
-		(end 91.75 55)
+		(start 88.96 86.96)
+		(end 88.96 86)
 		(width 1)
 		(layer "B.Cu")
@@
 	)
 	(segment
+		(start 98.25 78)
+		(end 91.75 78)
+		(width 1)
+		(layer "F.Cu")
+		(net 13)
+	)
+	(segment
 		(start 89 90.46)
 		(end 86.54 88)
@@
 	)
 	(segment
+		(start 48.75 55)
+		(end 55.25 55)
+		(width 1)
+		(layer "F.Cu")
+		(net 15)
+	)
+	(segment
 		(start 81.34 86)
 		(end 81.34 90.12)
@@
 	)
 	(segment
-		(start 52 58.25)
-		(end 48.75 55)
+		(start 52 78.25)
+		(end 52 59.375)
 		(width 1)
 		(layer "B.Cu")
@@
 	)
 	(segment
-		(start 81 90.46)
-		(end 80.46 91)
+		(start 64.75 91)
+		(end 52 78.25)
 		(width 1)
 		(layer "B.Cu")
@@
 	)
 	(segment
-		(start 64.75 91)
-		(end 52 78.25)
+		(start 52 59.375)
+		(end 48.75 56.125)
 		(width 1)
 		(layer "B.Cu")
@@
 	)
 	(segment
-		(start 52 78.25)
-		(end 52 58.25)
+		(start 48.75 56.125)
+		(end 48.75 55)
 		(width 1)
 		(layer "B.Cu")
@@
 	)
 	(segment
-		(start 80.46 91)
-		(end 64.75 91)
+		(start 81 90.46)
+		(end 80.46 91)
 		(width 1)
 		(layer "B.Cu")
@@
 	)
 	(segment
+		(start 80.46 91)
+		(end 64.75 91)
+		(width 1)
+		(layer "B.Cu")
+		(net 15)
+	)
+	(segment
+		(start 48.75 78)
+		(end 55.25 78)
+		(width 1)
+		(layer "F.Cu")
+		(net 16)
+	)
+	(segment
 		(start 82.25 93.5)
 		(end 63.5 93.5)
@@
 	)
 	(segment
+		(start 55.25 73.5)
+		(end 48.75 73.5)
+		(width 1)
+		(layer "F.Cu")
+		(net 19)
+	)
+	(segment
+		(start 98.25 59.5)
+		(end 91.75 59.5)
+		(width 1)
+		(layer "F.Cu")
+		(net 19)
+	)
+	(segment
+		(start 55.25 59.5)
+		(end 48.75 59.5)
+		(width 1)
+		(layer "F.Cu")
+		(net 19)
+	)
+	(segment
+		(start 91.75 73.5)
+		(end 98.25 73.5)
+		(width 1)
+		(layer "F.Cu")
+		(net 19)
+	)
+	(segment

Commit message: change psu, add some 3d
Parts:
- removed PS1: IRM-03-5, Converter_ACDC:Converter_ACDC_MeanWell_IRM-03-xx_THT
- added D1: 1N914, Diode_THT:D_DO-35_SOD27_P7.62mm_Horizontal, F.Cu at (38.0, 41.7)
- added D2: 1N914, Diode_THT:D_DO-35_SOD27_P7.62mm_Horizontal, F.Cu at (38.0, 36.8)
- added PS2: IRM-05-5, Converter_ACDC:Converter_ACDC_MeanWell_IRM-05-xx_THT, F.Cu at (74.5, 30.3)
- Q1, Q2: footprint Package_TO_SOT_THT:TO-92 -> Package_TO_SOT_THT:TO-92_Wide
- moved R1 12.9 mm to (83.5, 81.7)
- moved R2 12.9 mm to (79.5, 81.7)
- moved R3 12.9 mm to (71.5, 81.7)
- moved R4 12.9 mm to (75.5, 81.7)
- moved U1 11.2 mm to (73.0, 85.0)
- moved R5 4.62 mm to (46.5, 90.5)
- moved Q1 4.38 mm to (50.0, 85.4)
- moved R8 3.72 mm to (50.5, 95.5)
- moved Q2 2.91 mm to (41.3, 85.4)
- moved R6 2.88 mm to (37.5, 90.5)
- moved R7 2.18 mm to (41.5, 95.5)
- moved J1 1.73 mm to (41.6, 49.2)
- moved J2 1.73 mm to (41.6, 36.8)
Connections:
- J3 pad 2: /AC_SW2_L -> /AC_IN_L
- J3 pad 3: /AC_IN_L -> /AC_SW2_L
Routing:
- net +3V3: track 106.2 -> 72.7 mm
- net GND: track 140.8 -> 108.4 mm
- net /BTN4: track 56.0 -> 36.8 mm
- net /BTN3: track 70.2 -> 52.1 mm
- net /AC_IN_L: track 50.0 -> 67.2 mm
- net /AC_IN_N: track 47.8 -> 36.3 mm
- net /BTN1: track 53.0 -> 43.1 mm
- net /AC_SW2_L: track 45.8 -> 38.0 mm
- net /BTN2: track 23.6 -> 29.3 mm
- net /SW2: track 44.2 -> 39.6 mm
- net Net-(D1-A): track 54.2 -> 50.3 mm
- net /SW1: track 27.7 -> 24.1 mm
- net /AC_SW1_L: track 35.4 -> 36.9 mm
- net Net-(D2-A): track 65.0 -> 63.6 mm
- net +5V: track 93.2 -> 92.4 mm
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Other:
- board size 80 x 80 mm -> 80 x 75 mm

Commit message: idk hw or smth
Routing:
- net GND: track 108.4 -> 87.8 mm
- net /AC_IN_L: track 67.2 -> 68.1 mm
Changed lines of the file:
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@@
 	)
 	(segment
-		(start 85.5 44.5)
-		(end 82.9 41.9)
+		(start 86.5 44.5)
+		(end 85 43)
+		(width 3)
+		(layer "B.Cu")
+		(net 2)
+	)
+	(segment
+		(start 85 43)
+		(end 51.5 43)
+		(width 3)
+		(layer "B.Cu")
+		(net 2)
+	)
+	(segment
+		(start 51.5 43)
+		(end 49.001 40.501)
+		(width 3)
+		(layer "B.Cu")
+		(net 2)
+	)
+	(segment
+		(start 52.1 29.4)
+		(end 56.81 29.4)
+		(width 3)
+		(layer "B.Cu")
+		(net 2)
+	)
+	(segment
+		(start 56.81 29.4)
+		(end 62.8075 29.4)
 		(width 3)
 		(layer "B.Cu")
@@
 	)
 	(segment
-		(start 51.9 41.9)
-		(end 56.81 41.9)
-		(width 3)
-		(layer "B.Cu")
-		(net 2)
-	)
-	(segment
-		(start 49.001 32.499)
-		(end 49.001 39.001)
-		(width 3)
-		(layer "B.Cu")
-		(net 2)
-	)
-	(segment
-		(start 82.9 41.9)
-		(end 56.81 41.9)
-		(width 3)
-		(layer "B.Cu")
-		(net 2)
-	)
-	(segment
-		(start 49.001 39.001)
-		(end 51.9 41.9)
-		(width 3)
-		(layer "B.Cu")
-		(net 2)
-	)
-	(segment
-		(start 56.81 29.4)
-		(end 62.8075 29.4)
+		(start 49.001 40.501)
+		(end 49.001 32.499)
 		(width 3)
 		(layer "B.Cu")
@@
 	(segment
 		(start 91 44.5)
-		(end 85.5 44.5)
+		(end 86.5 44.5)
 		(width 3)
 		(layer "B.Cu")
@@
 	)
 	(segment
-		(start 52.1 29.4)
-		(end 56.81 29.4)
-		(width 3)
-		(layer "B.Cu")
-		(net 2)
-	)
-	(segment
 		(start 50.04 85.5)
 		(end 50.04 85.04)
@@
 		(net 7)
 	)
-	(segment
-		(start 63.61 74)
-		(end 64.11 74.5)
-		(width 1)
-		(layer "F.Cu")
-		(net 8)
-	)
-	(segment
-		(start 59 87.5)
-		(end 59 75.75)
-		(width 1)
-		(layer "F.Cu")
-		(net 8)
-	)
-	(segment
-		(start 57 89.5)
-		(end 59 87.5)
-		(width 1)
-		(layer "F.Cu")
-		(net 8)
-	)
-	(segment
-		(start 59 75.75)
-		(end 60.75 74)
-		(width 1)
-		(layer "F.Cu")
-		(net 8)
-	)
-	(segment
-		(start 60.75 74)
-		(end 63.61 74)
-		(width 1)
-		(layer "F.Cu")
-		(net 8)
-	)
 	(via
