File: SmartyB-hw/SmartyB-hw.kicad_sch (KiCad schematic)
At the start: 3 parts, among them J1 1-2071556-2, J2 1-2071556-2

Commit message: some moar hw stuff
Parts:
- added J3, J4: Screw_Terminal_01x03, TerminalBlock_RND:TerminalBlock_RND_205-00046_1x03_P5.00mm_Horizontal, symbol Connector:Screw_Terminal_01x03
- added Q1, Q2: Q_NMOS_DGS, Package_TO_SOT_THT:TO-92, symbol Transistor_FET:Q_NMOS_DGS
- added R1, R2, R3, R4: 10K, Resistor_THT:R_Axial_DIN0204_L3.6mm_D1.6mm_P5.08mm_Horizontal, symbol Device:R
- added R5, R6: 100K, Resistor_THT:R_Axial_DIN0204_L3.6mm_D1.6mm_P5.08mm_Horizontal, symbol Device:R
- added R7, R8: 1K, Resistor_THT:R_Axial_DIN0204_L3.6mm_D1.6mm_P5.08mm_Horizontal, symbol Device:R
- added SW1, SW2, SW3, SW4: SW_Push, Button_Switch_THT:SW_PUSH_6mm_H5mm, symbol Switch:SW_Push
- added U1: ~, SmartyB:ESP32_C6_SUPERMINI, symbol SmartyB:ESP32_C6_SUPERMINI
Connections:
- net +5V: now reaches J1.1 (COIL_1)
- net +5V: now also J2.1 (COIL_1), PS1.16 (+Vo), U1.11 (5V)
- net at J1.2 (COIL_2): now also Q1.1 (D)
- net AC_SW1_L: now reaches J1.3 (COM)
- net AC_SW1_L: now also J3.1 (Pin_1)
- net AC_IN_L: now reaches J1.4 (NO)
- net AC_IN_L: now also J2.4 (NO), PS1.1 (AC/L), J3.3 (Pin_3)
- net GND: now reaches PS1.14 (-Vo)
- net GND: now also Q1.3 (S), Q2.3 (S), R1.2, R2.2, R3.2, R4.2, R5.2, R6.2, U1.12 (GND)
- net AC_IN_N: now reaches PS1.3 (AC/N)
- net AC_IN_N: now also J4.1 (Pin_1), J4.2 (Pin_2), J4.3 (Pin_3)
- net at J2.2 (COIL_2): now also Q2.1 (D)
- net AC_SW2_L: now reaches J2.3 (COM)
- net AC_SW2_L: now also J3.2 (Pin_2)
- new net: Q1.2 (G), R5.1, R8.2
- new net: Q2.2 (G), R6.1, R7.2
- new net +3V3: SW1.1, SW2.1, SW3.1, SW4.1, U1.13 (3V3)
- new net BTN1: R1.1, SW1.2, U1.19 (GP9)
- new net BTN2: R2.1, SW2.2, U1.18 (GP14)
- new net BTN3: R3.1, SW3.2, U1.16 (GP18)
- new net BTN4: R4.1, SW4.2, U1.17 (GP15)
- new net SW1: R8.1, U1.5 (GP2)
- new net SW2: R7.1, U1.6 (GP3)
Other:
- moved on the sheet: J1, J2

Commit message: change psu, add some 3d
Parts:
- removed PS1: IRM-03-5, Converter_ACDC:Converter_ACDC_MeanWell_IRM-03-xx_THT, symbol Converter_ACDC:IRM-03-5
- added D1, D2: 1N914, Diode_THT:D_DO-35_SOD27_P7.62mm_Horizontal, symbol Diode:1N914
- added PS2: IRM-05-5, Converter_ACDC:Converter_ACDC_MeanWell_IRM-05-xx_THT, symbol Converter_ACDC:IRM-05-5
Connections:
- net +5V: now also D1.1 (K), D2.1 (K), PS2.4 (+Vo)
- net AC_IN_L: now also J3.2 (Pin_2), PS2.2 (AC/L); no longer J3.3 (Pin_3)
- net AC_IN_N: now also PS2.1 (AC/N)
- net AC_SW2_L: now also J3.3 (Pin_3); no longer J3.2 (Pin_2)
- net GND: now also PS2.3 (-Vo)
- net at J1.2 (COIL_2), Q1.1 (D): now also D1.2 (A)
- net at J2.2 (COIL_2), Q2.1 (D): now also D2.2 (A)

Commit message: readme + kicad10
Parts:
- U1: value ~ -> (none)
